File: Hardware/Schematic.sch (EAGLE design)
At the start: 103 parts, among them IC1 BD5229G-TR, IC4 XC6220A331MR-G, J1 FH34SRJ-24S-0.5SH_99_, J2 SAMACSYS_PARTS_USB4110-GF-A, J3 QWIIC_RIGHT_ANGLE, J4 112A-TAAR-R03_ATTEND, Q1 20V/4.2A/52mΩ/1.4W, Q2 20V/4.2A/52mΩ/1.4W, Q3 SI1308EDL-T1-GE3, U1 W25Q512JVEIQ, U2 ESP32-C6-WROOM-1-N8, U3 DS3231SN#, U4 MAX17048G+T10

Commit message: Resolved the raised issues
Other:
- note removed: "OpenBook Schematic"
Changed lines of the file:
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@@
 <text x="1054.1" y="-426.72" size="2.54" layer="97">External NOR Flash 64MB</text>
 <text x="1089.66" y="-464.82" size="2.54" layer="94">drawn by: Rafael Chitan</text>
-<text x="1038.86" y="-472.44" size="2.54" layer="94">OpenBook Schematic</text>
 </plain>
 <instances>
@@
 <segment>
 <wire x1="1097.28" y1="-299.72" x2="1099.82" y2="-299.72" width="0.1524" layer="91"/>
-<label x="1099.82" y="-299.72" size="1.778" layer="95" xref="yes"/>
+<label x="1099.82" y="-299.72" size="1.27" layer="95" xref="yes"/>
 <pinref part="U2" gate="G$1" pin="IO12"/>
 </segment>
@@
 <segment>
 <wire x1="1097.28" y1="-302.26" x2="1099.82" y2="-302.26" width="0.1524" layer="91"/>
-<label x="1099.82" y="-302.26" size="1.778" layer="95" xref="yes"/>
+<label x="1099.82" y="-302.26" size="1.27" layer="95" xref="yes"/>
 <pinref part="U2" gate="G$1" pin="IO13"/>
 </segment>
@@
 <segment>
 <wire x1="1056.64" y1="-309.88" x2="1054.1" y2="-309.88" width="0.1524" layer="91"/>
-<label x="1054.1" y="-309.88" size="1.778" layer="95" rot="R180" xref="yes"/>
+<label x="1054.1" y="-309.88" size="1.27" layer="95" rot="R180" xref="yes"/>
 <pinref part="U2" gate="G$1" pin="IO4"/>
 </segment>
@@
 <segment>
 <wire x1="1056.64" y1="-317.5" x2="1054.1" y2="-317.5" width="0.1524" layer="91"/>
-<label x="1054.1" y="-317.5" size="1.778" layer="95" rot="R180" xref="yes"/>
+<label x="1054.1" y="-317.5" size="1.27" layer="95" rot="R180" xref="yes"/>
 <pinref part="U2" gate="G$1" pin="IO7"/>
 </segment>
@@
 <segment>
 <wire x1="1056.64" y1="-304.8" x2="1054.1" y2="-304.8" width="0.1524" layer="91"/>
-<label x="1054.1" y="-304.8" size="1.778" layer="95" rot="R180" xref="yes"/>
+<label x="1054.1" y="-304.8" size="1.27" layer="95" rot="R180" xref="yes"/>
 <pinref part="U2" gate="G$1" pin="IO2"/>
 </segment>
@@
 <segment>
 <wire x1="1056.64" y1="-314.96" x2="1054.1" y2="-314.96" width="0.1524" layer="91"/>
-<label x="1054.1" y="-314.96" size="1.778" layer="95" rot="R180" xref="yes"/>
+<label x="1054.1" y="-314.96" size="1.27" layer="95" rot="R180" xref="yes"/>
 <pinref part="U2" gate="G$1" pin="IO6"/>
 </segment>
@@
 <segment>
 <wire x1="1056.64" y1="-294.64" x2="1054.1" y2="-294.64" width="0.1524" layer="91"/>
-<label x="1054.1" y="-294.64" size="1.778" layer="95" rot="R180" xref="yes"/>
+<label x="1054.1" y="-294.64" size="1.27" layer="95" rot="R180" xref="yes"/>
 <pinref part="U2" gate="G$1" pin="EN"/>
 </segment>
@@
 <segment>
 <wire x1="1056.64" y1="-299.72" x2="1054.1" y2="-299.72" width="0.1524" layer="91"/>
-<label x="1054.1" y="-299.72" size="1.778" layer="95" rot="R180" xref="yes"/>
+<label x="1054.1" y="-299.72" size="1.27" layer="95" rot="R180" xref="yes"/>
 <pinref part="U2" gate="G$1" pin="IO0"/>
 </segment>
@@
 <segment>
 <wire x1="1056.64" y1="-302.26" x2="1054.1" y2="-302.26" width="0.1524" layer="91"/>
-<label x="1054.1" y="-302.26" size="1.778" layer="95" rot="R180" xref="yes"/>
+<label x="1054.1" y="-302.26" size="1.27" layer="95" rot="R180" xref="yes"/>
 <pinref part="U2" gate="G$1" pin="IO1"/>
 </segment>
@@
 <segment>
 <wire x1="1056.64" y1="-307.34" x2="1054.1" y2="-307.34" width="0.1524" layer="91"/>
-<label x="1054.1" y="-307.34" size="1.778" layer="95" rot="R180" xref="yes"/>
+<label x="1054.1" y="-307.34" size="1.27" layer="95" rot="R180" xref="yes"/>
 <pinref part="U2" gate="G$1" pin="IO3"/>
 </segment>
@@
 <segment>
 <wire x1="1056.64" y1="-312.42" x2="1054.1" y2="-312.42" width="0.1524" layer="91"/>
-<label x="1054.1" y="-312.42" size="1.778" layer="95" rot="R180" xref="yes"/>
+<label x="1054.1" y="-312.42" size="1.27" layer="95" rot="R180" xref="yes"/>
 <pinref part="U2" gate="G$1" pin="IO5"/>
 </segment>
@@
 <segment>
 <wire x1="1097.28" y1="-325.12" x2="1099.82" y2="-325.12" width="0.1524" layer="91"/>
-<label x="1099.82" y="-325.12" size="1.778" layer="95" xref="yes"/>
+<label x="1099.82" y="-325.12" size="1.27" layer="95" xref="yes"/>
 <pinref part="U2" gate="G$1" pin="IO23"/>
 </segment>
@@
 <segment>
 <wire x1="1097.28" y1="-322.58" x2="1099.82" y2="-322.58" width="0.1524" layer="91"/>
-<label x="1099.82" y="-322.58" size="1.778" layer="95" xref="yes"/>
+<label x="1099.82" y="-322.58" size="1.27" layer="95" xref="yes"/>
 <pinref part="U2" gate="G$1" pin="IO22"/>
 </segment>
@@
 <segment>
 <wire x1="1097.28" y1="-320.04" x2="1099.82" y2="-320.04" width="0.1524" layer="91"/>
-<label x="1099.82" y="-320.04" size="1.778" layer="95" xref="yes"/>
+<label x="1099.82" y="-320.04" size="1.27" layer="95" xref="yes"/>
 <pinref part="U2" gate="G$1" pin="IO21"/>
 </segment>
@@
 <segment>
 <wire x1="1097.28" y1="-317.5" x2="1099.82" y2="-317.5" width="0.1524" layer="91"/>
-<label x="1099.82" y="-317.5" size="1.778" layer="95" xref="yes"/>
+<label x="1099.82" y="-317.5" size="1.27" layer="95" xref="yes"/>
 <pinref part="U2" gate="G$1" pin="IO20"/>
 </segment>
@@
 <segment>
 <wire x1="1097.28" y1="-314.96" x2="1099.82" y2="-314.96" width="0.1524" layer="91"/>
-<label x="1099.82" y="-314.96" size="1.778" layer="95" xref="yes"/>
+<label x="1099.82" y="-314.96" size="1.27" layer="95" xref="yes"/>
 <pinref part="U2" gate="G$1" pin="IO19"/>
 </segment>
@@
 <segment>
 <wire x1="1097.28" y1="-312.42" x2="1099.82" y2="-312.42" width="0.1524" layer="91"/>
-<label x="1099.82" y="-312.42" size="1.778" layer="95" xref="yes"/>
+<label x="1099.82" y="-312.42" size="1.27" layer="95" xref="yes"/>
 <pinref part="U2" gate="G$1" pin="IO18"/>
 </segment>
@@
 <segment>
 <wire x1="1097.28" y1="-309.88" x2="1099.82" y2="-309.88" width="0.1524" layer="91"/>
-<label x="1099.82" y="-309.88" size="1.778" layer="95" xref="yes"/>
+<label x="1099.82" y="-309.88" size="1.27" layer="95" xref="yes"/>
 <pinref part="U2" gate="G$1" pin="RXD0/GPIO17"/>
 </segment>
@@
 <segment>
 <wire x1="1097.28" y1="-307.34" x2="1099.82" y2="-307.34" width="0.1524" layer="91"/>
-<label x="1099.82" y="-307.34" size="1.778" layer="95" xref="yes"/>
+<label x="1099.82" y="-307.34" size="1.27" layer="95" xref="yes"/>
 <pinref part="U2" gate="G$1" pin="TXD0/GPIO16"/>
 </segment>
@@
 <segment>
 <wire x1="1097.28" y1="-304.8" x2="1099.82" y2="-304.8" width="0.1524" layer="91"/>
-<label x="1099.82" y="-304.8" size="1.778" layer="95" xref="yes"/>
+<label x="1099.82" y="-304.8" size="1.27" layer="95" xref="yes"/>
 <pinref part="U2" gate="G$1" pin="IO15"/>
 </segment>
@@
 <segment>
 <wire x1="1097.28" y1="-297.18" x2="1099.82" y2="-297.18" width="0.1524" layer="91"/>
-<label x="1099.82" y="-297.18" size="1.778" layer="95" xref="yes"/>
+<label x="1099.82" y="-297.18" size="1.27" layer="95" xref="yes"/>
 <pinref part="U2" gate="G$1" pin="IO11"/>
 </segment>
@@
 <segment>
 <wire x1="1097.28" y1="-294.64" x2="1099.82" y2="-294.64" width="0.1524" layer="91"/>
-<label x="1099.82" y="-294.64" size="1.778" layer="95" xref="yes"/>
+<label x="1099.82" y="-294.64" size="1.27" layer="95" xref="yes"/>
 <pinref part="U2" gate="G$1" pin="IO10"/>
 </segment>
@@
 </sheet>
 </sheets>
+<errors>
+</errors>
 </schematic>
 </drawing>
